File: Ebow_experimental_smt/Ebow.kicad_pcb (KiCad board)
At the start: 2 copper layers, 53.8 x 29 mm, 11 parts, among them J1 Conn_01x02, U1 LM386

Commit message: added inductor part number (SMNR6028-4R7MT)
Parts:
- L1, L2: value L_Iron -> SMNR6028-4R7MT
Connections:
- net +5V renamed +9V
Changed lines of the file:
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@@
   (net 5 "Net-(C3-Pad1)")
   (net 6 "Net-(C3-Pad2)")
-  (net 7 "+5V")
+  (net 7 "+9V")
   (net 8 "Net-(C4-Pad2)")
   (net 9 "Net-(L1-Pad2)")
@@
     (descr "Through hole straight pin header, 1x02, 2.54mm pitch, single row")
     (tags "Through hole pin header THT 1x02 2.54mm single row")
-    (property "Sheetfile" "Ebow.kicad_sch")
+    (property "Sheetfile" "File: Ebow.kicad_sch")
     (property "Sheetname" "")
     (attr through_hole)
@@
     (fp_line (start -1.27 3.81) (end -1.27 -0.635) (layer "F.Fab") (width 0.1))
     (pad "1" thru_hole rect (at 0 0 180) (size 1.7 1.7) (drill 1) (layers *.Cu *.Mask)
-      (net 7 "+5V") (pinfunction "Pin_1") (pintype "passive"))
+      (net 7 "+9V") (pinfunction "Pin_1") (pintype "passive"))
     (pad "2" thru_hole oval (at 0 2.54 180) (size 1.7 1.7) (drill 1) (layers *.Cu *.Mask)
       (net 2 "GND") (pinfunction "Pin_2") (pintype "passive"))
@@
     (descr "SOIC, 8 Pin (JEDEC MS-012AA, https://www.analog.com/media/en/package-pcb-resources/package/pkg_pdf/soic_narrow-r/r_8.pdf), generated with kicad-footprint-generator ipc_gullwing_generator.py")
     (tags "SOIC SO")
-    (property "Sheetfile" "Ebow.kicad_sch")
+    (property "Sheetfile" "File: Ebow.kicad_sch")
     (property "Sheetname" "")
     (attr smd)
@@
       (net 6 "Net-(C3-Pad2)") (pintype "output"))
     (pad "6" smd roundrect (at 2.475 0.635) (size 1.95 0.6) (layers "F.Cu" "F.Paste" "F.Mask") (roundrect_rratio 0.25)
-      (net 7 "+5V") (pinfunction "V+") (pintype "power_in"))
+      (net 7 "+9V") (pinfunction "V+") (pintype "power_in"))
     (pad "7" smd roundrect (at 2.475 -0.635) (size 1.95 0.6) (layers "F.Cu" "F.Paste" "F.Mask") (roundrect_rratio 0.25)
       (net 4 "/BYPASS1") (pinfunction "BYPASS") (pintype "input"))
@@
     (descr "SMD capacitor, aluminum electrolytic nonpolar, 4.0x5.8mm")
     (tags "capacitor electrolyic nonpolar")
-    (property "Sheetfile" "Ebow.kicad_sch")
+    (property "Sheetfile" "File: Ebow.kicad_sch")
     (property "Sheetname" "")
     (attr smd)
@@
     (descr "Mounting Hole 2.5mm")
     (tags "mounting hole 2.5mm")
-    (property "Sheetfile" "Ebow.kicad_sch")
+    (property "Sheetfile" "File: Ebow.kicad_sch")
     (property "Sheetname" "")
     (attr exclude_from_pos_files)
@@
     (descr "Resistor SMD 0805 (2012 Metric), square (rectangular) end terminal, IPC_7351 nominal with elongated pad for handsoldering. (Body size source: IPC-SM-782 page 72, https://www.pcb-3d.com/wordpress/wp-content/uploads/ipc-sm-782a_amendment_1_and_2.pdf), generated with kicad-footprint-generator")
     (tags "resistor handsolder")
-    (property "Sheetfile" "Ebow.kicad_sch")
+    (property "Sheetfile" "File: Ebow.kicad_sch")
     (property "Sheetname" "")
     (attr smd)
@@
     (descr "Inductor, Taiyo Yuden, NR series, Taiyo-Yuden_NR-80xx, 8.0mmx8.0mm")
     (tags "inductor taiyo-yuden nr smd")
-    (property "Sheetfile" "Ebow.kicad_sch")
+    (property "Sheetfile" "File: Ebow.kicad_sch")
     (property "Sheetname" "")
     (attr smd)
@@
       (effects (font (size 1 1) (thickness 0.15)))
     )
-    (fp_text value "L_Iron" (at 0 5.5 90) (layer "F.Fab")
+    (fp_text value "SMNR6028-4R7MT" (at 0 5.5 90) (layer "F.Fab")
       (effects (font (size 1 1) (thickness 0.15)))
     )
@@
     (descr "SMD capacitor, aluminum electrolytic nonpolar, 4.0x5.8mm")
     (tags "capacitor electrolyic nonpolar")
-    (property "Sheetfile" "Ebow.kicad_sch")
+    (property "Sheetfile" "File: Ebow.kicad_sch")
     (property "Sheetname" "")
     (attr smd)
@@
     (descr "SMD capacitor, aluminum electrolytic, Panasonic E7, 8.0x6.9mm")
     (tags "capacitor electrolytic")
-    (property "Sheetfile" "Ebow.kicad_sch")
+    (property "Sheetfile" "File: Ebow.kicad_sch")
     (property "Sheetname" "")
     (attr smd)
@@
     (descr "Capacitor SMD 0805 (2012 Metric), square (rectangular) end terminal, IPC_7351 nominal with elongated pad for handsoldering. (Body size source: IPC-SM-782 page 76, https://www.pcb-3d.com/wordpress/wp-content/uploads/ipc-sm-782a_amendment_1_and_2.pdf, https://docs.google.com/spreadsheets/d/1BsfQQcO9C6DZCsRaXUlFlo91Tg2WpOkGARC1WS5S8t0/edit?usp=sharing), generated with kicad-footprint-generator")
     (tags "capacitor handsolder")
-    (property "Sheetfile" "Ebow.kicad_sch")
+    (property "Sheetfile" "File: Ebow.kicad_sch")
     (property "Sheetname" "")
     (attr smd)
@@
     (descr "Mounting Hole 2.5mm")
     (tags "mounting hole 2.5mm")
-    (property "Sheetfile" "Ebow.kicad_sch")
+    (property "Sheetfile" "File: Ebow.kicad_sch")
     (property "Sheetname" "")
     (attr exclude_from_pos_files)
@@
     (descr "Inductor, Taiyo Yuden, NR series, Taiyo-Yuden_NR-80xx, 8.0mmx8.0mm")
     (tags "inductor taiyo-yuden nr smd")
-    (property "Sheetfile" "Ebow.kicad_sch")
+    (property "Sheetfile" "File: Ebow.kicad_sch")
     (property "Sheetname" "")
     (attr smd)
@@
       (effects (font (size 1 1) (thickness 0.15)))
     )
-    (fp_text value "L_Iron" (at 0 5.5 90) (layer "F.Fab")
-      (effects (font (size 1 1) (thickness 0.15)))
-    )
+    (fp_text value "SMNR6028-4R7MT" (at 0 5.5 90) (layer "F.Fab")
+      (effects (font (size 1 1) (thickness 0.15)))
+    )
